Commit message: feat: add link to sensors.xacro

File: sensor_kit/data_collection_car_sensor_kit_launch/data_collection_car_sensor_kit_description/urdf/sensors.xacro (robot description, xacro)
@@ -4,4 +4,5 @@
   <xacro:property name="calibration" value="${xacro.load_yaml('$(arg config_dir)/sensors_calibration.yaml')}"/>
   <xacro:include filename="sensor_kit.xacro"/>
+  <link name="base_link"/>
   <xacro:sensor_kit_macro
     parent="base_link"
